File: breakout.kicad_pcb (KiCad board)
At the start: 2 copper layers, 50 x 50 mm, 25 parts, among them J1 JACK_TRS_4PINS, P1 CONN_01X08, P2 SPEAKER, P3 ISO7816_SIMPLE, P4 CONN_01X09, P5 SMA_CONN, P6 CONN_01X02, P7 USB_A, Q1 Q_PMOS_GSD, Q2 Q_NMOS_GSD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

Commit message: Add a bunch of audio crap.
Parts:
- removed G***: LOGO, Stochastic:Logo_5mm
- added C1: 33uF, Capacitors_SMD:C_0805_HandSoldering, F.Cu at (176.8, 93.2)
- added C10: 33uF, Capacitors_SMD:C_0805_HandSoldering, F.Cu at (176.8, 83.0)
- added C11: 33uF, Capacitors_SMD:C_0805_HandSoldering, F.Cu at (176.8, 88.1)
- added C5: 33uF, Capacitors_SMD:C_0805_HandSoldering, F.Cu at (179.3, 93.2)
- added C6: 10uF, Capacitors_SMD:C_0805_HandSoldering, F.Cu at (176.8, 78.0)
- added C7: 10uF, Capacitors_SMD:C_0805_HandSoldering, F.Cu at (179.3, 83.0)
- added C8: 10uF, Capacitors_SMD:C_0805_HandSoldering, F.Cu at (179.3, 88.1)
- added C9: 33uF, Capacitors_SMD:C_0805_HandSoldering, F.Cu at (179.3, 78.0)
- added LOGO: LOGO, Stochastic:Logo_5mm, F.Cu at (193.1, 96.9)
- added R8: 68Ω, Resistors_SMD:R_0805_HandSoldering, F.Cu at (178.1, 97.0)
- P6: value CONN_01X02 -> MIC
- moved P6 4.59 mm to (187.4, 79.4), turned to 270 degrees
- moved J1 1.80 mm to (186.1, 91.9)
Connections:
- net /GPIO12 renamed /ESP_TX
- net /GPIO14 renamed /ESP_RX
- GSM1 pad 21: /MIC+ -> /MIC2_P
- J1 pad 5: /MIC+ -> Net-(C5-Pad1)
Routing:
- net /MIC+: track 26.1 -> 0.00 mm
- net Net-(C5-Pad1): track 0.00 -> 22.7 mm
- net /EARL: track 11.4 -> 27.3 mm, vias 0 -> 2
- net GND: track 42.7 -> 54.6 mm, vias 3 -> 4
- net /MIC2_P: track 0.00 -> 11.4 mm
- net /GPIO2: track 35.7 -> 39.5 mm
- net Net-(GSM1-Pad20): track 39.7 -> 43.4 mm
- net /PWRCTL: track 53.4 -> 57.0 mm
- net /GPIO0: track 32.1 -> 34.6 mm
- net /ESP_RX: track 38.4 -> 40.2 mm
- net /EARR: track 18.7 -> 20.4 mm
- net /GPIO4: track 20.5 -> 22.1 mm
- net /RX: track 13.8 -> 15.4 mm
- net /TX: track 10.4 -> 12.0 mm
- net /ESP_TX: track 35.3 -> 34.3 mm
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Other:
- board text added: "JUST LOOK AT THE SCHEMATIC, I CAN'T EVEN"
