File: breakout.sch (KiCad schematic (older format))
At the start: 37 parts, among them J1 JACK_TRS_4PINS, P1 CONN_01X08, P2 SPEAKER, P3 ISO7816_SIMPLE, P4 CONN_01X09, P5 SMA_CONN, P6 MIC, P7 USB_OTG, Q1 Q_PMOS_GSD, Q2 Q_NMOS_GSD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

Commit message: Change A6 TX/RX pins.
Connections:
- net GPIO16 is gone; now on net ESP_RX: P4.4 (P4), U2.4 (GPIO16)
- net ESP_RX: no longer P4.5 (P5), U2.5 (GPIO14)
- net ESP_TX: now also P4.5 (P5), U2.5 (GPIO14); no longer P4.6 (P6), U2.6 (GPIO12)
- net VCC renamed Vcc
- new net GPIO12: P4.6 (P6), U2.6 (GPIO12)
Changed lines of the file:
@@
 L PWR_FLAG #FLG01
 U 1 1 57ADD23B
-P 10200 6150
-F 0 "#FLG01" H 10200 6245 50  0001 C CNN
-F 1 "PWR_FLAG" H 10200 6330 50  0000 C CNN
-F 2 "" H 10200 6150 50  0000 C CNN
-F 3 "" H 10200 6150 50  0000 C CNN
-	1    10200 6150
+P 11000 6200
+F 0 "#FLG01" H 11000 6295 50  0001 C CNN
+F 1 "PWR_FLAG" H 11000 6380 50  0000 C CNN
+F 2 "" H 11000 6200 50  0000 C CNN
+F 3 "" H 11000 6200 50  0000 C CNN
+	1    11000 6200
 	1    0    0    -1
 $EndComp
@@
 L GND #PWR02
 U 1 1 57ADD255
-P 10200 6300
-F 0 "#PWR02" H 10200 6050 50  0001 C CNN
-F 1 "GND" H 10200 6150 50  0000 C CNN
-F 2 "" H 10200 6300 50  0000 C CNN
-F 3 "" H 10200 6300 50  0000 C CNN
-	1    10200 6300
-	1    0    0    -1
-$EndComp
-$Comp
-L PWR_FLAG #FLG03
-U 1 1 57ADD285
-P 10700 6150
-F 0 "#FLG03" H 10700 6245 50  0001 C CNN
-F 1 "PWR_FLAG" H 10700 6330 50  0000 C CNN
-F 2 "" H 10700 6150 50  0000 C CNN
-F 3 "" H 10700 6150 50  0000 C CNN
-	1    10700 6150
+P 11000 6350
+F 0 "#PWR02" H 11000 6100 50  0001 C CNN
+F 1 "GND" H 11000 6200 50  0000 C CNN
+F 2 "" H 11000 6350 50  0000 C CNN
+F 3 "" H 11000 6350 50  0000 C CNN
+	1    11000 6350
 	1    0    0    -1
 $EndComp
@@
 $EndComp
 $Comp
-L GND #PWR04
+L GND #PWR03
 U 1 1 57AFB015
 P 5350 3350
-F 0 "#PWR04" H 5350 3100 50  0001 C CNN
+F 0 "#PWR03" H 5350 3100 50  0001 C CNN
 F 1 "GND" H 5358 3176 50  0000 C CNN
 F 2 "" H 5350 3350 50  0000 C CNN
@@
 $EndComp
 $Comp
-L GND #PWR05
+L GND #PWR04
 U 1 1 57B03856
 P 6250 5750
-F 0 "#PWR05" H 6250 5500 50  0001 C CNN
+F 0 "#PWR04" H 6250 5500 50  0001 C CNN
 F 1 "GND" H 6250 5600 50  0000 C CNN
 F 2 "" H 6250 5750 50  0000 C CNN
@@
 $EndComp
 $Comp
-L GND #PWR06
+L GND #PWR05
 U 1 1 57B076AE
 P 5800 6950
-F 0 "#PWR06" H 5800 6700 50  0001 C CNN
+F 0 "#PWR05" H 5800 6700 50  0001 C CNN
 F 1 "GND" H 5800 6800 50  0000 C CNN
 F 2 "" H 5800 6950 50  0000 C CNN
@@
 $EndComp
 $Comp
-L GND #PWR07
+L GND #PWR06
 U 1 1 57B4FD98
 P 2500 6100
-F 0 "#PWR07" H 2500 5850 50  0001 C CNN
+F 0 "#PWR06" H 2500 5850 50  0001 C CNN
 F 1 "GND" H 2500 5950 50  0000 C CNN
 F 2 "" H 2500 6100 50  0000 C CNN
@@
 NoConn ~ 2100 1400
 $Comp
-L VCC #PWR08
-U 1 1 57B52833
-P 11050 6150
-F 0 "#PWR08" H 11050 6000 50  0001 C CNN
-F 1 "VCC" H 11050 6300 50  0000 C CNN
-F 2 "" H 11050 6150 50  0000 C CNN
-F 3 "" H 11050 6150 50  0000 C CNN
-	1    11050 6150
-	1    0    0    -1
-$EndComp
-$Comp
-L VCC #PWR09
-U 1 1 57B52878
-P 1100 1150
-F 0 "#PWR09" H 1100 1000 50  0001 C CNN
-F 1 "VCC" H 1100 1300 50  0000 C CNN
-F 2 "" H 1100 1150 50  0000 C CNN
-F 3 "" H 1100 1150 50  0000 C CNN
-	1    1100 1150
-	1    0    0    -1
-$EndComp
-$Comp
-L VCC #PWR010
-U 1 1 57B52AB7
-P 10400 1150
-F 0 "#PWR010" H 10400 1000 50  0001 C CNN
-F 1 "VCC" H 10400 1300 50  0000 C CNN
-F 2 "" H 10400 1150 50  0000 C CNN
-F 3 "" H 10400 1150 50  0000 C CNN
-	1    10400 1150
-	1    0    0    -1
-$EndComp
-$Comp
 L CONN_01X08 P1
 U 1 1 57B52EB3
@@
 $EndComp
 $Comp
-L GND #PWR011
+L GND #PWR07
 U 1 1 57B7110B
 P 9950 2150
-F 0 "#PWR011" H 9950 1900 50  0001 C CNN
+F 0 "#PWR07" H 9950 1900 50  0001 C CNN
 F 1 "GND" H 9950 2000 50  0000 C CNN
 F 2 "" H 9950 2150 50  0000 C CNN
@@
 $EndComp
 $Comp
-L GND #PWR012
+L GND #PWR08
 U 1 1 57BA1E9B
 P 10700 2850
-F 0 "#PWR012" H 10700 2600 50  0001 C CNN
+F 0 "#PWR08" H 10700 2600 50  0001 C CNN
 F 1 "GND" H 10700 2700 50  0000 C CNN
 F 2 "" H 10700 2850 50  0000 C CNN
@@
 $EndComp
 $Comp
-L GND #PWR013
+L GND #PWR09
 U 1 1 57BA8917
 P 8600 4150
-F 0 "#PWR013" H 8600 3900 50  0001 C CNN
+F 0 "#PWR09" H 8600 3900 50  0001 C CNN
 F 1 "GND" H 8600 4000 50  0000 C CNN
 F 2 "" H 8600 4150 50  0000 C CNN
@@
 $EndComp
 $Comp
-L GND #PWR014
+L GND #PWR010
 U 1 1 57BA8BFB
 P 9100 3500
-F 0 "#PWR014" H 9100 3250 50  0001 C CNN
+F 0 "#PWR010" H 9100 3250 50  0001 C CNN
 F 1 "GND" H 9100 3350 50  0000 C CNN
 F 2 "" H 9100 3500 50  0000 C CNN
@@
 Text Label 5850 6100 0    60   ~ 0
 ESP_RX
-Text Label 3000 3200 1    60   ~ 0
+Text Label 3000 3100 1    60   ~ 0
 ESP_RX
-Text Label 2900 3200 1    60   ~ 0
+Text Label 2900 3100 1    60   ~ 0
 ESP_TX
 Wire Wire Line
-	10200 6150 10200 6300
-Wire Wire Line
-	10700 6150 10700 6250
-Wire Wire Line
-	10700 6250 11050 6250
-Wire Wire Line
-	11050 6250 11050 6150
+	11000 6200 11000 6350
 Wire Wire Line
 	2550 2050 3250 2050
@@
 Wire Wire Line
 	2550 2350 3250 2350
-Connection ~ 3000 2450
-Connection ~ 2900 2550
 Wire Wire Line
 	2550 2650 3250 2650
@@
 Connection ~ 9000 3500
 Wire Wire Line
-	3000 3200 3000 2450
-Wire Wire Line
-	2900 3200 2900 2550
+	3000 3100 3000 2350
+Wire Wire Line
+	2900 3100 2900 2450
 Wire Wire Line
 	5550 6100 5850 6100
@@
 	7800 3900 7800 4000
 $Comp
-L GND #PWR015
+L GND #PWR011
 U 1 1 57BAEA0B
 P 7700 3950
-F 0 "#PWR015" H 7700 3700 50  0001 C CNN
+F 0 "#PWR011" H 7700 3700 50  0001 C CNN
 F 1 "GND" H 7700 3800 50  0000 C CNN
 F 2 "" H 7700 3950 50  0000 C CNN
@@
 Connection ~ 7800 3950
 $Comp
-L GND #PWR016
+L GND #PWR012
 U 1 1 57BAEB9B
 P 7700 5050
-F 0 "#PWR016" H 7700 4800 50  0001 C CNN
+F 0 "#PWR012" H 7700 4800 50  0001 C CNN
 F 1 "GND" H 7700 4900 50  0000 C CNN
 F 2 "" H 7700 5050 50  0000 C CNN
@@
 Connection ~ 1650 3100
 Wire Wire Line
-	1100 1150 1100 3300
+	1100 1250 1100 3300
 NoConn ~ 1400 3300
+Connection ~ 3000 2350
+Connection ~ 2900 2450
+Text Label 10400 1150 1    60   ~ 0
+Vcc
+Text Label 1100 3250 1    60   ~ 0
+Vcc
 $EndSCHEMATC

Commit message: Fix capacitor values
Parts:
- C1, C10, C11, C5, C9: value 33uF -> 33pF
- C6, C7, C8: value 10uF -> 10pF
- D1: symbol LED -> LED-RESCUE-breakout
- P7: symbol USB_OTG -> USB_OTG-RESCUE-breakout
- U1: symbol APE8865Y5-31-HF-3 -> APE8865Y5-31-HF-3-RESCUE-breakout
Changed lines of the file:
@@
 EESchema Schematic File Version 2
+LIBS:breakout-rescue
 LIBS:power
 LIBS:device
@@
 $EndComp
 $Comp
-L APE8865Y5-31-HF-3 U1
+L APE8865Y5-31-HF-3-RESCUE-breakout U1
 U 1 1 57B514AD
 P 1650 1300
@@
 GPIO13
 $Comp
-L LED D1
+L LED-RESCUE-breakout D1
 U 1 1 57BA1DA8
 P 10700 2150
@@
 P 8750 3300
 F 0 "C1" H 8800 3400 50  0000 L CNN
-F 1 "33uF" H 8550 3200 50  0000 L CNN
+F 1 "33pF" H 8550 3200 50  0000 L CNN
 F 2 "Capacitors_SMD:C_0805_HandSoldering" H 8865 3208 50  0001 L CNN
 F 3 "" H 8750 3300 50  0000 C CNN
@@
 P 8750 3700
 F 0 "C5" H 8800 3800 50  0000 L CNN
-F 1 "33uF" H 8550 3600 50  0000 L CNN
+F 1 "33pF" H 8550 3600 50  0000 L CNN
 F 2 "Capacitors_SMD:C_0805_HandSoldering" H 8865 3608 50  0001 L CNN
 F 3 "" H 8750 3700 50  0000 C CNN
@@
 P 8200 4550
 F 0 "C7" H 8250 4650 50  0000 L CNN
-F 1 "10uF" H 8250 4450 50  0000 L CNN
+F 1 "10pF" H 8250 4450 50  0000 L CNN
 F 2 "Capacitors_SMD:C_0805_HandSoldering" H 8315 4458 50  0001 L CNN
 F 3 "" H 8200 4550 50  0000 C CNN
@@
 P 7800 4550
 F 0 "C10" H 7850 4650 50  0000 L CNN
-F 1 "33uF" H 7850 4450 50  0000 L CNN
+F 1 "33pF" H 7850 4450 50  0000 L CNN
 F 2 "Capacitors_SMD:C_0805_HandSoldering" H 7915 4458 50  0001 L CNN
 F 3 "" H 7800 4550 50  0000 C CNN
@@
 P 8200 4150
 F 0 "C6" H 8250 4250 50  0000 L CNN
-F 1 "10uF" H 8250 4050 50  0000 L CNN
+F 1 "10pF" H 8250 4050 50  0000 L CNN
 F 2 "Capacitors_SMD:C_0805_HandSoldering" H 8315 4058 50  0001 L CNN
 F 3 "" H 8200 4150 50  0000 C CNN
@@
 P 7800 4150
 F 0 "C9" H 7850 4250 50  0000 L CNN
-F 1 "33uF" H 7850 4050 50  0000 L CNN
+F 1 "33pF" H 7850 4050 50  0000 L CNN
 F 2 "Capacitors_SMD:C_0805_HandSoldering" H 7915 4058 50  0001 L CNN
 F 3 "" H 7800 4150 50  0000 C CNN
@@
 P 7800 4900
 F 0 "C11" H 7850 5000 50  0000 L CNN
-F 1 "33uF" H 7850 4800 50  0000 L CNN
+F 1 "33pF" H 7850 4800 50  0000 L CNN
 F 2 "Capacitors_SMD:C_0805_HandSoldering" H 7915 4808 50  0001 L CNN
 F 3 "" H 7800 4900 50  0000 C CNN
@@
 P 8200 4900
 F 0 "C8" H 8250 5000 50  0000 L CNN
-F 1 "10uF" H 8250 4800 50  0000 L CNN
+F 1 "10pF" H 8250 4800 50  0000 L CNN
 F 2 "Capacitors_SMD:C_0805_HandSoldering" H 8315 4808 50  0001 L CNN
 F 3 "" H 8200 4900 50  0000 C CNN
@@
 	6250 6500 6350 6500
 $Comp
-L USB_OTG P7
+L USB_OTG-RESCUE-breakout P7
 U 1 1 57DB372C
 P 1300 3600
